Commit message: 追加

File: urdf/simple_robot.urdf.xacro (robot description, xacro)
@@ -67,4 +67,23 @@
         </inertial>
     </link>
+    <link name="camera_link">
+        <visual>
+            <geometry>
+                <box size="0.05 0.05 0.05"/>
+            </geometry>
+            <material name="red">
+                <color rgba="1.0 0.0 0.0 1.0"/>
+            </material>
+        </visual>
+        <collision>
+            <geometry>
+                <box size="0.05 0.05 0.05"/>
+            </geometry>
+        </collision>
+        <inertial>
+            <mass value="0.1"/>
+            <inertia ixx="0.0001" ixy="0.0" ixz="0.0" iyy="0.0001" iyz="0.0" izz="0.0001"/>
+        </inertial>
+    </link>
     <joint name="base_footprint_joint" type="fixed">
         <parent link="base_footprint"/>
@@ -83,4 +102,9 @@
         <origin xyz="${base_length/4} ${wheel_separation/2} ${-base_height/2}" rpy="0 0 0"/>
         <axis xyz="0 1 0"/>
+    </joint>
+    <joint name="camera_joint" type="fixed">
+        <parent link="base_link"/>
+        <child link="camera_link"/>
+        <origin xyz="${base_length/2} 0 ${base_height/2 + 0.02}" rpy="0 0 0"/>
     </joint>
     <ros2_control name="GazeboSystem" type="system">
@@ -105,3 +129,25 @@
         </plugin>
     </gazebo>
+    <gazebo reference="camera_link">
+        <plugin name="camera_controller" filename="libgazebo_ros_camera.so">
+            <ros>
+                <namespace>/camera</namespace>
+                <image_topic>image_raw</image_topic>
+                <camera_info_topic>camera_info</camera_info_topic>
+            </ros>
+            <camera name="my_camera">
+                <horizontal_fov>1.396</horizontal_fov>
+                <image>
+                    <width>640</width>
+                    <height>480</height>
+                    <format>R8G8B8</format>
+                </image>
+                <clip>
+                    <near>0.02</near>
+                    <far>300</far>
+                </clip>
+            </camera>
+            <update_rate>30.0</update_rate>
+        </plugin>
+    </gazebo>
 </robot>
